File: pcb_files/kicad_project/IRTimer.kicad_pcb (KiCad board)
At the start: 6 copper layers, 50 x 47 mm, 39 parts, among them J1 Conn_01x02_Pin, J2 Conn_01x02_Pin, SW1 SW_DPDT_x2, U1 TSOP382xx

Commit message: Corrige gambada en el routeo de SCL y SDA de la TFT
Parts:
- removed SENSOR: ~, Connector_PinHeader_2.54mm:PinHeader_1x03_P2.54mm_Vertical
- added S1: ~, Connector_PinHeader_2.54mm:PinHeader_1x03_P2.54mm_Vertical, F.Cu at (136.2, 88.1)
- moved G*** 1.00 mm to (134.9, 93.0)
- moved G*** 0.92 mm to (133.0, 92.4)
- moved MODE 0.17 mm to (156.1, 87.7)
- moved RESET 0.07 mm to (156.1, 99.6)
Connections:
- ESP1 pad 4: /TFT_MOSI -> /TFT_SDA
- ESP1 pad 5: /TFT_SCLK -> /TFT_SCL
- LCD1 pad 3: /TFT_SCLK -> /TFT_SCL
- LCD1 pad 4: /TFT_SCLK -> /TFT_SDA
Routing:
- net /TFT_SDA: track 0.00 -> 51.1 mm, vias 0 -> 1
- net /TFT_SCLK: track 42.9 -> 0.00 mm, vias 1 -> 0
- net /TFT_SCL: track 0.00 -> 42.2 mm, vias 0 -> 1
- net +3V3: track 166.7 -> 171.7 mm
