File: pcb_files/kicad_project/IRTimer.kicad_sch (KiCad schematic)
At the start: 25 parts, among them J1 Conn_01x02_Pin, J2 Conn_01x02_Pin, SW1 SW_DPDT_x2, U1 TSOP382xx

Commit message: Corrige gambada en el routeo de SCL y SDA de la TFT
Connections:
- net TFT_MOSI renamed TFT_SDA
- net TFT_SDA: now also LCD1.4 (SDA)
- net TFT_SCLK renamed TFT_SCL
- net TFT_SCL: no longer LCD1.4 (SDA)
Changed lines of the file:
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@@
+	(wire
+		(pts
+			(xy 114.3 154.94) (xy 104.14 154.94)
+		)
+		(stroke
+			(width 0)
+			(type default)
+		)
+	)
 	(wire
 		(pts
@@
 		(pts
 			(xy 179.07 121.92) (xy 193.04 121.92)
-		)
-		(stroke
-			(width 0)
-			(type default)
-		)
-	)
-	(wire
-		(pts
-			(xy 114.3 154.94) (xy 104.14 154.94)
 		)
 		(stroke
@@
 		)
 	)
-	(label "TFT_SCLK"
+	(label "TFT_SCL"
+		(at 114.3 154.94 180)
+		(fields_autoplaced yes)
+		(effects
+			(font
+				(size 1.27 1.27)
+			)
+			(justify right bottom)
+		)
+	)
+	(label "TFT_SCL"
 		(at 116.84 50.8 0)
 		(fields_autoplaced yes)
@@
 			)
 			(justify left bottom)
+		)
+	)
+	(label "TFT_SDA"
+		(at 114.3 157.48 180)
+		(fields_autoplaced yes)
+		(effects
+			(font
+				(size 1.27 1.27)
+			)
+			(justify right bottom)
 		)
 	)
@@
 		)
 	)
-	(label "TFT_SCLK"
-		(at 114.3 157.48 180)
-		(fields_autoplaced yes)
-		(effects
-			(font
-				(size 1.27 1.27)
-			)
-			(justify right bottom)
-		)
-	)
 	(label "BATT"
 		(at 250.19 82.55 180)
@@
 		)
 	)
-	(label "TFT_SCLK"
-		(at 114.3 154.94 180)
-		(fields_autoplaced yes)
-		(effects
-			(font
-				(size 1.27 1.27)
-			)
-			(justify right bottom)
-		)
-	)
 	(label "TFT_RES"
 		(at 166.37 48.26 180)
@@
 		)
 	)
-	(label "TFT_MOSI"
+	(label "TFT_SDA"
 		(at 116.84 48.26 0)
 		(fields_autoplaced yes)
@@
 			)
 		)
-		(property "Description" ""
+		(property "Description" "Multiple-cell battery"
 			(at 185.42 147.32 0)
 			(effects
@@
 			)
 		)
-		(property "Description" ""
+		(property "Description" "Switch, dual pole double throw, separate symbols"
 			(at 184.15 116.84 0)
 			(effects
